Commit message: pangolin_simulation.launch.py: 修改默认仿真赛道为有墙赛道，并保留无墙赛道选项。 mid360.xacro: 修正激光雷达模型参数，通过model:从模型库加载的方式报错但是能够显示雷达外观。通过packages:从功能包加载方式未报错但是加载速度很慢，容易加载不出来。

File: src/simulation_environment/rc_robot_simulation/livox_laser_simulation_RO2/install/ros2_livox_simulation/share/ros2_livox_simulation/urdf/mid360.xacro (robot description, xacro)
@@ -25,4 +25,5 @@
         <geometry>
           <mesh filename="model://mid360.stl" scale="0.0008 0.0008 0.0008"/>
+          <!-- <mesh filename="package://pangolin_simulation/meshes/mid360.stl" scale="0.0008 0.0008 0.0008"/> -->
         </geometry>
       </visual>
