Commit message: 针对R2机器人导航系统的调试与优化工作已完成核心功能验证，其中r2_bringup功能包下的启动配置文件经修改后，系统主体导航与定位模块可稳定运行；但在坐标系变换（TF）链路验证中发现，当前系统仅能有效发布map→odom的全局坐标变换关系，关键的odom→base_link局部坐标变换链路存在缺失。也就是fastlivo的里程计没有使用上，无法满足导航系统对定位精度的需求。结合系统开发历程追溯分析可知，该问题的核心诱因在于系统里程计模块由Fast-LIO迁移至Fast-LIVO的过程中，Fast-LIO原本具备的odom→base_link坐标变换发布配置规则未在Fast-LIVO中同步保留，导致机器人局部运动信息与全局定位信息的传递链路中断，进而影响导航系统的完整运行。

File: src/simulation_environment/rc_robot_simulation/pangolin_simulation/install/pangolin_simulation/share/pangolin_simulation/urdf/real_waking_robot.xacro (robot description, xacro)
@@ -1,144 +1 @@
-<?xml version="1.0"?>
-<robot name="robot" xmlns:xacro="http://www.ros.org/wiki/xacro">
-    <xacro:property name="length_wheel" value="0.05" />
-    <xacro:property name="radius_wheel" value="0.06" />
-    <xacro:property name="PI" value="3.1415926"/>
-    <xacro:macro name="default_inertial" params="mass">
-        <inertial>
-            <mass value="${mass}" />
-            <inertia ixx="0.01" ixy="0.0" ixz="0.0"
-                    iyy="0.01" iyz="0.0" izz="0.01" />
-        </inertial>
-    </xacro:macro>
-    <link name="base_link">
-        <visual>
-            <geometry>
-                <box size="0.2 .3 .1"/>
-            </geometry>
-            <origin rpy="0 0 ${PI/2}" xyz="0 0 0.05"/>
-            <material name="white">
-                <color rgba="1 1 1 1"/>
-            </material>
-        </visual>
-        <collision>
-            <geometry>
-                <box size="0.2 .3 0.1"/>
-            </geometry>
-            <origin rpy="0 0 ${PI/2}" xyz="0 0 0.05"/>
-        </collision>
-        <xacro:default_inertial mass="8.2"/>
-    </link>
-    <link name="wheel_1">
-        <visual>
-            <geometry>
-                <cylinder length="${length_wheel}" radius="${radius_wheel}"/>
-            </geometry>
-            <origin rpy="0 0 0" xyz="0 0 0"/>
-            <material name="black">
-                <color rgba="0 0 0 1"/>
-            </material>
-        </visual>
-        <collision>
-            <geometry>
-                <cylinder length="${length_wheel}" radius="${radius_wheel}"/>
-            </geometry>
-        </collision>
-        <mu1>0.5</mu1>
-        <mu2>0.5</mu2>
-        <xacro:default_inertial mass="0.5"/>
-    </link>
-    <link name="wheel_2">
-        <visual>
-            <geometry>
-                <cylinder length="${length_wheel}" radius="${radius_wheel}"/>
-            </geometry>
-            <origin rpy="0 0 0" xyz="0 0 0"/>
-            <material name="black"/>
-        </visual>
-        <collision>
-            <geometry>
-                <cylinder length="${length_wheel}" radius="${radius_wheel}"/>
-            </geometry>
-        </collision>
-        <mu1>0.5</mu1>
-        <mu2>0.5</mu2>
-        <xacro:default_inertial mass="0.5"/>
-    </link>
-    <link name="wheel_3">
-        <visual>
-            <geometry>
-                <cylinder length="${length_wheel}" radius="${radius_wheel}"/>
-            </geometry>
-            <origin rpy="0 0 0" xyz="0 0 0"/>
-            <material name="black"/>
-        </visual>
-        <collision>
-            <geometry>
-                <cylinder length="${length_wheel}" radius="${radius_wheel}"/>
-            </geometry>
-        </collision>
-        <mu1>0.5</mu1>
-        <mu2>0.5</mu2>
-        <xacro:default_inertial mass="0.5"/>
-    </link>
-    <link name="wheel_4">
-        <visual>
-            <geometry>
-                <cylinder length="${length_wheel}" radius="${radius_wheel}"/>
-            </geometry>
-            <origin rpy="0 0 0" xyz="0 0 0" />
-            <material name="black"/>
-        </visual>
-        <collision>
-            <geometry>
-                <cylinder length="${length_wheel}" radius="${radius_wheel}"/>
-            </geometry>
-        </collision>
-        <mu1>0.5</mu1>
-        <mu2>0.5</mu2>
-        <xacro:default_inertial mass="0.5"/>
-    </link>
-    <joint name="base_to_wheel1" type="continuous">
-        <parent link="base_link"/>
-        <child link="wheel_1"/>
-        <origin rpy="${-PI/2} 0 0" xyz="0.1 0.13 0"/>
-        <axis xyz="0 0 1" />
-    </joint>
-    <joint name="base_to_wheel2" type="continuous">
-        <axis xyz="0 0 1" />
-        <anchor xyz="0 0 0" />
-        <limit effort="100" velocity="100" />
-        <parent link="base_link"/>
-        <child link="wheel_2"/>
-        <origin rpy="${-PI/2} 0 0" xyz="-0.1 0.13 0"/>
-    </joint>
-    <joint name="base_to_wheel3" type="continuous">
-        <parent link="base_link"/>
-        <axis xyz="0 0 1" />
-        <child link="wheel_3"/>
-        <origin rpy="${-PI/2} 0 0" xyz="0.1 -0.13 0"/>
-    </joint>
-    <joint name="base_to_wheel4" type="continuous">
-        <parent link="base_link"/>
-        <axis xyz="0 0 1" />
-        <child link="wheel_4"/>
-        <origin rpy="${-PI/2} 0 0" xyz="-0.1 -0.13 0"/>
-    </joint>
-    <!-- Livox-Mid360  -->
-    <link name="livox_frame">
-        <visual>
-            <origin xyz="0.025 -0.0265 -0.025" rpy="${pi/2} 0 ${pi}"/>
-            <geometry>
-                <mesh filename="package://pb_rm_simulation/meshes/mid360.stl" scale="0.001 0.001 0.001"/>
-            </geometry>
-            <material name="blue">
-                <color rgba="0 0 1.0 1" />
-            </material>
-        </visual>
-    </link>
-    <joint name="livox_joint" type="fixed">
-        <origin xyz="0 0.0 0.17" rpy="0 0 0"/>
-        <parent link="base_link"/>
-        <child link="livox_frame"/>
-    </joint>
-</robot>
+/home/oh/SCURC_Nav_Sim/src/simulation_environment/rc_robot_simulation/pangolin_simulation/urdf/real_waking_robot.xacro

File: src/simulation_environment/rc_robot_simulation/pangolin_simulation/install/pangolin_simulation/share/pangolin_simulation/urdf/simulation_waking_robot.xacro (robot description, xacro)
@@ -1,234 +1 @@
-<?xml version="1.0"?>
-<robot name="robot" xmlns:xacro="http://www.ros.org/wiki/xacro">
-    <xacro:property name="length_wheel" value="0.05" />
-    <xacro:property name="radius_wheel" value="0.06" />
-    <xacro:property name="PI" value="3.1415926"/>
-    <xacro:macro name="default_inertial" params="mass">
-        <inertial>
-            <mass value="${mass}" />
-            <inertia ixx="0.01" ixy="0.0" ixz="0.0"
-                    iyy="0.01" iyz="0.0" izz="0.01" />
-        </inertial>
-    </xacro:macro>
-    <link name="base_link">
-        <visual>
-            <geometry>
-                <box size="0.2 .3 .1"/>
-            </geometry>
-            <origin rpy="0 0 ${PI/2}" xyz="0 0 0.05"/>
-            <material name="white">
-                <color rgba="1 1 1 1"/>
-            </material>
-        </visual>
-        <collision>
-            <geometry>
-                <box size="0.2 .3 0.1"/>
-            </geometry>
-            <origin rpy="0 0 ${PI/2}" xyz="0 0 0.05"/>
-        </collision>
-        <xacro:default_inertial mass="8.2"/>
-    </link>
-    <link name="yaw_link"/>
-    <joint name="base_to_yaw" type="continuous">
-        <parent link="base_link"/>
-        <child link="yaw_link"/>
-        <origin rpy="0 0 0" xyz="0 0 0.1"/>
-        <axis xyz="0 0 1" />
-    </joint>
-    <link name="wheel_1">
-        <visual>
-            <geometry>
-                <cylinder length="${length_wheel}" radius="${radius_wheel}"/>
-            </geometry>
-            <origin rpy="0 0 0" xyz="0 0 0"/>
-            <material name="black">
-                <color rgba="0 0 0 1"/>
-            </material>
-        </visual>
-        <collision>
-            <geometry>
-                <cylinder length="${length_wheel}" radius="${radius_wheel}"/>
-            </geometry>
-        </collision>
-        <mu1>0.5</mu1>
-        <mu2>0.5</mu2>
-        <xacro:default_inertial mass="0.5"/>
-    </link>
-    <link name="wheel_2">
-        <visual>
-            <geometry>
-                <cylinder length="${length_wheel}" radius="${radius_wheel}"/>
-            </geometry>
-            <origin rpy="0 0 0" xyz="0 0 0"/>
-            <material name="black"/>
-        </visual>
-        <collision>
-            <geometry>
-                <cylinder length="${length_wheel}" radius="${radius_wheel}"/>
-            </geometry>
-        </collision>
-        <mu1>0.5</mu1>
-        <mu2>0.5</mu2>
-        <xacro:default_inertial mass="0.5"/>
-    </link>
-    <link name="wheel_3">
-        <visual>
-            <geometry>
-                <cylinder length="${length_wheel}" radius="${radius_wheel}"/>
-            </geometry>
-            <origin rpy="0 0 0" xyz="0 0 0"/>
-            <material name="black"/>
-        </visual>
-        <collision>
-            <geometry>
-                <cylinder length="${length_wheel}" radius="${radius_wheel}"/>
-            </geometry>
-        </collision>
-        <mu1>0.5</mu1>
-        <mu2>0.5</mu2>
-        <xacro:default_inertial mass="0.5"/>
-    </link>
-    <link name="wheel_4">
-        <visual>
-            <geometry>
-                <cylinder length="${length_wheel}" radius="${radius_wheel}"/>
-            </geometry>
-            <origin rpy="0 0 0" xyz="0 0 0" />
-            <material name="black"/>
-        </visual>
-        <collision>
-            <geometry>
-                <cylinder length="${length_wheel}" radius="${radius_wheel}"/>
-            </geometry>
-        </collision>
-        <mu1>0.5</mu1>
-        <mu2>0.5</mu2>
-        <xacro:default_inertial mass="0.5"/>
-    </link>
-    <joint name="base_to_wheel1" type="continuous">
-        <parent link="base_link"/>
-        <child link="wheel_1"/>
-        <origin rpy="${-PI/2} 0 0" xyz="0.1 0.13 0"/>
-        <axis xyz="0 0 1" />
-    </joint>
-    <joint name="base_to_wheel2" type="continuous">
-        <axis xyz="0 0 1" />
-        <anchor xyz="0 0 0" />
-        <parent link="base_link"/>
-        <child link="wheel_2"/>
-        <origin rpy="${-PI/2} 0 0" xyz="-0.1 0.13 0"/>
-    </joint>
-    <joint name="base_to_wheel3" type="continuous">
-        <parent link="base_link"/>
-        <axis xyz="0 0 1" />
-        <child link="wheel_3"/>
-        <origin rpy="${-PI/2} 0 0" xyz="0.1 -0.13 0"/>
-    </joint>
-    <joint name="base_to_wheel4" type="continuous">
-        <parent link="base_link"/>
-        <axis xyz="0 0 1" />
-        <child link="wheel_4"/>
-        <origin rpy="${-PI/2} 0 0" xyz="-0.1 -0.13 0"/>
-    </joint>
-    <!-- IMU joint -->
-    <joint name="imu_joint" type="fixed">
-        <axis xyz="0 1 0" />
-        <origin xyz="0 0 0.125" rpy="0 0 0"/>
-        <parent link="base_link"/>
-        <child link="imu_link"/>
-    </joint>
-    <!-- IMU -->
-    <link name="imu_link">
-        <collision>
-            <origin xyz="0 0 0" rpy="0 0 0"/>
-            <geometry>
-                <box size="0.05 0.05 0.05"/>
-            </geometry>
-        </collision>
-        <visual>
-            <origin xyz="0 0 0" rpy="0 0 0"/>
-            <geometry>
-                <box size="0.05 0.05 0.05"/>
-            </geometry>
-            <material name="green">
-                <color rgba="0 1 0 1"/>
-            </material>
-        </visual>
-        <inertial>
-            <mass value="1e-2" />
-            <origin xyz="0 0 0" rpy="0 0 0"/>
-            <inertia ixx="1e-6" ixy="0" ixz="0" iyy="1e-6" iyz="0" izz="1e-6" />
-        </inertial>
-    </link>
-    <!-- gazebo插件设置相关 -->
-    <gazebo reference="base_link">
-        <material>Gazebo/Orange</material>
-    </gazebo>
-    <gazebo reference="wheel_1">
-        <material>Gazebo/Red</material>
-    </gazebo>
-    <gazebo reference="wheel_2">
-        <material>Gazebo/Black</material>
-    </gazebo>
-    <gazebo reference="wheel_3">
-        <material>Gazebo/Red</material>
-    </gazebo>
-    <gazebo reference="wheel_4">
-        <material>Gazebo/Black</material>
-    </gazebo>
-    <!-- Drive controller -->
-    <gazebo>
-        <plugin name="mecanum_controller" filename="libcmd_vel_z_plugin.so">
-        <!-- <plugin name="mecanum_controller" filename="libgazebo_ros_planar_move.so"> -->
-            <ros>
-                <!-- <namespace>/demo</namespace> -->
-                <remapping>cmd_vel:=cmd_vel</remapping>
-                <remapping>odom:=state_estimation</remapping>
-            </ros>
-            <update_rate>20</update_rate>
-            <publish_rate>20</publish_rate>
-            <publish_odom>false</publish_odom>
-            <publish_odom_tf>false</publish_odom_tf>
-            <odometry_frame>odom</odometry_frame>
-            <robot_base_frame>base_link</robot_base_frame>
-        </plugin>
-    </gazebo>
-    <!-- imu控制 -->
-    <gazebo reference="imu_link">
-        <material>Gazebo/Orange</material>
-        <gravity>false</gravity>
-        <sensor name="imu_sensor" type="imu">
-            <always_on>true</always_on>
-            <update_rate>200</update_rate>
-            <!-- 关键：开启重力补偿，即使Gazebo无重力，也让IMU输出模拟重力的z轴加速度 -->
-            <!-- <gravity_compensation>true</gravity_compensation> -->
-            <!-- 手动设置模拟重力的加速度（z轴向下为负，对应-9.8m/s²） -->
-            <!-- <xacro:property name="sim_gravity_z" value="-9.8" /> -->
-            <!-- <linear_acceleration_bias>0 0 ${sim_gravity_z}</linear_acceleration_bias> -->
-            <visualize>true</visualize>
-            <topic>__default_topic__</topic>
-            <plugin filename="libgazebo_ros_imu_sensor.so" name="imu_plugin">
-                <topicName>/livox/imu</topicName>
-                <bodyName>imu_link</bodyName>
-                <updateRateHZ>100.0</updateRateHZ>
-                <gaussianNoise>0.0</gaussianNoise>
-                <xyzOffset>0 0 0</xyzOffset>
-                <rpyOffset>0 0 0</rpyOffset>
-                <frameName>imu_link</frameName>
-                <serviceName>default_service</serviceName>
-                <alwaysOn>true</alwaysOn>
-                <maxAngularVelocity>100.0</maxAngularVelocity>
-                <noiseDensity>0.0</noiseDensity>
-                <randomWalk>0.0</randomWalk>
-                <ros>
-                    <remapping>~/out:=/livox/imu</remapping>
-                </ros>
-            </plugin>
-        </sensor>
-    </gazebo>
-    <!-- Livox-Mid360  -->
-    <xacro:include filename="$(find ros2_livox_simulation)/urdf/mid360.xacro" />
-    <xacro:mid360 name="livox_frame" parent="base_link" topic="/livox/lidar">
-        <origin xyz="0 0.0 0.175" rpy="0 0 0"/>
-    </xacro:mid360>
-</robot>
+/home/oh/SCURC_Nav_Sim/src/simulation_environment/rc_robot_simulation/pangolin_simulation/urdf/simulation_waking_robot.xacro
