Commit message: 删除了build log install文件

File: src/simulation_environment/rc_robot_simulation/install/pangolin_simulation/share/pangolin_simulation/urdf/simulation_waking_robot.xacro (robot description, xacro)
@@ -161,4 +161,30 @@
         </inertial>
     </link>
+    <link name="camera_link">
+        <visual>
+        <geometry>
+            <box size="0.04 0.04 0.04"/>
+        </geometry>
+        <material name="blue">
+            <color rgba="0 0 1 1"/>
+        </material>
+    </visual>
+    <collision>
+        <geometry>
+            <box size="0.04 0.04 0.04"/>
+        </geometry>
+    </collision>
+        <inertial>
+        <mass value="0.05"/>
+            <inertia ixx="1e-5" ixy="0" ixz="0"
+                 iyy="1e-5" iyz="0"
+                 izz="1e-5"/>
+        </inertial>
+    </link>
+    <joint name="camera_joint" type="fixed">
+    <parent link="base_link"/>
+    <child link="camera_link"/>
+    <origin xyz="0.15 0 0.18" rpy="0 0 0"/>
+    </joint>
     <!-- gazebo插件设置相关 -->
     <gazebo reference="base_link">
@@ -227,4 +253,32 @@
         </sensor>
     </gazebo>
+    <gazebo reference="camera_link">
+    <sensor name="camera_sensor" type="camera">
+        <always_on>true</always_on>
+        <update_rate>30</update_rate>
+        <visualize>true</visualize>
+        <camera>
+            <horizontal_fov>1.047</horizontal_fov>
+            <image>
+                <width>640</width>
+                <height>480</height>
+                <format>R8G8B8</format>
+            </image>
+            <clip>
+                <near>0.05</near>
+                <far>50</far>
+            </clip>
+        </camera>
+        <plugin name="gazebo_ros_camera" filename="libgazebo_ros_camera.so">
+            <ros>
+                <namespace>/camera</namespace>
+            </ros>
+            <camera_name>front_camera</camera_name>
+            <frame_name>camera_link</frame_name>
+            <image_topic_name>image_raw</image_topic_name>
+            <camera_info_topic_name>camera_info</camera_info_topic_name>
+        </plugin>
+    </sensor>
+    </gazebo>
     <!-- Livox-Mid360  -->
     <xacro:include filename="$(find ros2_livox_simulation)/urdf/mid360.xacro" />
