Commit message: 加入yolo_ros2_ws的yolov8_ros2包，包含YOLOv8目标检测功能及相关配置和启动文件，解析数据，后续解析数据发布每个标号格子对应KFS类型。下一步加入根据解析数据规划路径。以及KFS自动摆放脚本。

File: src/simulation_environment/rc_robot_simulation/pangolin_simulation/urdf/simulation_waking_robot.xacro (robot description, xacro)
@@ -163,29 +163,69 @@
     <link name="camera_link">
         <visual>
-        <geometry>
-            <box size="0.04 0.04 0.04"/>
-        </geometry>
-        <material name="blue">
-            <color rgba="0 0 1 1"/>
-        </material>
-    </visual>
-    <collision>
-        <geometry>
-            <box size="0.04 0.04 0.04"/>
-        </geometry>
-    </collision>
+            <geometry>
+                <box size="0.04 0.04 0.04"/>
+            </geometry>
+            <material name="blue">
+                <color rgba="0 0 1 1"/>
+            </material>
+        </visual>
+        <collision>
+            <geometry>
+                <box size="0.04 0.04 0.04"/>
+            </geometry>
+        </collision>
         <inertial>
-        <mass value="0.05"/>
-            <inertia ixx="1e-5" ixy="0" ixz="0"
-                 iyy="1e-5" iyz="0"
-                 izz="1e-5"/>
+            <mass value="0.05"/>
+            <inertia ixx="1e-5" ixy="0" ixz="0" iyy="1e-5" iyz="0" izz="1e-5"/>
         </inertial>
     </link>
     <joint name="camera_joint" type="fixed">
-    <parent link="base_link"/>
-    <child link="camera_link"/>
-    <origin xyz="0.15 0 0.18" rpy="0 0 0"/>
+        <parent link="base_link"/>
+        <child link="camera_link"/>
+        <origin xyz="0.15 0 0.18" rpy="0 0 0"/>
+    </joint>
+    <link name="camera_color_optical_frame"/>
+    <joint name="camera_optical_joint" type="fixed">
+        <parent link="camera_link"/>
+        <child link="camera_color_optical_frame"/>
+        <origin xyz="0 0 0" rpy="-1.5708 0 -1.5708"/>
     </joint>
     <!-- gazebo插件设置相关 -->
+    <!-- camera -->
+    <gazebo reference="camera_link">
+        <sensor name="camera_sensor" type="depth">
+            <always_on>true</always_on>
+            <update_rate>30</update_rate>
+            <visualize>true</visualize>
+            <camera>
+                <horizontal_fov>1.047</horizontal_fov>
+                <image>
+                    <width>640</width>
+                    <height>480</height>
+                    <format>R8G8B8</format>
+                </image>
+                <clip>
+                    <near>0.05</near>
+                    <far>50</far>
+                </clip>
+            </camera>
+            <plugin name="front_camera_controller" filename="libgazebo_ros_camera.so">
+                <ros>
+                    <namespace>/camera</namespace>
+                    <remapping>/camera/camera/image_raw:=/camera/camera/color/image_raw</remapping>
+                    <remapping>/camera/camera/camera_info:=/camera/camera/color/camera_info</remapping>
+                    <remapping>/camera/camera/depth/image_raw:=/camera/camera/aligned_depth_to_color/image_raw</remapping>
+                    <remapping>/camera/camera/depth/camera_info:=/camera/camera/aligned_depth_to_color/camera_info</remapping>
+                    <remapping>/camera/camera/points:=/camera/camera/depth/color/points</remapping>
+                </ros>
+                <camera_name>camera</camera_name>
+                <frame_name>camera_color_optical_frame</frame_name>
+                <hack_baseline>0.07</hack_baseline>
+                <min_depth>0.05</min_depth>
+                <max_depth>10.0</max_depth>
+            </plugin>
+        </sensor>
+    </gazebo>
+    <!-- camera end -->
     <gazebo reference="base_link">
         <material>Gazebo/Orange</material>
@@ -220,4 +260,5 @@
         </plugin>
     </gazebo>
+    <!-- Drive controller end -->
     <!-- imu控制 -->
     <gazebo reference="imu_link">
@@ -253,32 +294,5 @@
         </sensor>
     </gazebo>
-    <gazebo reference="camera_link">
-    <sensor name="camera_sensor" type="camera">
-        <always_on>true</always_on>
-        <update_rate>30</update_rate>
-        <visualize>true</visualize>
-        <camera>
-            <horizontal_fov>1.047</horizontal_fov>
-            <image>
-                <width>640</width>
-                <height>480</height>
-                <format>R8G8B8</format>
-            </image>
-            <clip>
-                <near>0.05</near>
-                <far>50</far>
-            </clip>
-        </camera>
-        <plugin name="gazebo_ros_camera" filename="libgazebo_ros_camera.so">
-            <ros>
-                <namespace>/camera</namespace>
-            </ros>
-            <camera_name>front_camera</camera_name>
-            <frame_name>camera_link</frame_name>
-            <image_topic_name>image_raw</image_topic_name>
-            <camera_info_topic_name>camera_info</camera_info_topic_name>
-        </plugin>
-    </sensor>
-    </gazebo>
+    <!-- IMU end -->
     <!-- Livox-Mid360  -->
     <xacro:include filename="$(find ros2_livox_simulation)/urdf/mid360.xacro" />
